Commit message: add e0509

File: doosan_robot/m0609.urdf (robot description, URDF)
Before this commit: robot m0609, 12 links, 11 joints
Links:
- link base_0: mass 3.722 -> 2.722
- link link2: geometry collision mesh filename=package://meshes/MF0609_2_0.dae scale=0.001 0.001 0.001; collision mesh filename=package://meshes/MF0609_2_1.dae scale=0.001 0.001 0.001
- link link4: geometry collision mesh filename=package://meshes/MF0609_4_0.dae scale=0.001 0.001 0.001; collision mesh filename=package://meshes/MF0609_4_1.dae scale=0.001 0.001 0.001
